File: Hardware/Electroturn.kicad_pcb (KiCad board)
At the start: 2 copper layers, 100 x 100 mm, 31 parts, among them J1 Encoder Terminal, J2 Stepper Motor Terminal, J3 Screw_Terminal_01x02, SW1 Feed Switch, SW2 Motor Braking Switch, SW3 Mode Right Scroll, SW4 Mode Left Scroll, SW5 Function Btn 1, SW6 Function Btn 2, SW7 Function Btn 2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

Commit message: Locking major control panel UI components
Parts:
- A1, C1, C2, J1, J2, J3, R1, R10, R11, R2, R3, R4, R5, R6, R7, R8, R9, U1, U2, U3: moved to B.Cu
- moved R2 256.4 mm to (260.2, 291.4), turned to 180 degrees
- moved R4 256.4 mm to (260.2, 286.3), turned to 180 degrees
- moved R10 248.1 mm to (277.9, 291.3), turned to 180 degrees
- moved R5 243.0 mm to (247.4, 278.6), turned to 180 degrees
- moved R1 240.3 mm to (243.6, 286.3), turned to 180 degrees
- moved R3 227.2 mm to (257.6, 271.0), turned to 180 degrees
- moved A1 221.2 mm to (172.9, 229.4), turned to 180 degrees
- moved U3 220.5 mm to (273.6, 273.0), turned to 180 degrees
- moved U2 220.2 mm to (219.4, 262.1), turned to 180 degrees
- moved R6 216.5 mm to (239.8, 265.9), turned to 180 degrees
- moved R7 216.5 mm to (239.8, 271.0), turned to 180 degrees
- moved R11 214.4 mm to (270.3, 255.8), turned to 180 degrees
- moved J1 211.6 mm to (202.9, 286.7), turned to 180 degrees
- moved J2 211.6 mm to (202.9, 278.6), turned to 180 degrees
- moved C1 210.1 mm to (274.1, 264.3), turned to 180 degrees
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Other:
- board size 100 x 100 mm -> 133.4 x 82.5 mm
